File: projects/ctrl-board/scheme/ctrl-board.sch (KiCad schematic (older format))
At the start: 54 parts

Commit message: Design...
Parts:
- removed C? (x2): 10u, symbol C
- removed K? (x3): i2c-1, symbol CONN_3
- removed R? (x5): 100, symbol R
- removed R? (x2): 50, symbol R
- removed R?: 10k, symbol R
- added C? (x4): C, symbol C
- added C? (x3): CP1, symbol CP1
- added D? (x2): DIODESCH, symbol DIODESCH
- added D?: 1N5819, symbol DIODESCH
- added D?: AD8607, symbol AD8607
- added K?: CONN_3, symbol CONN_3
- added K?: i2c-1, symbol CONN_3
- added L? (x2): INDUCTOR, symbol INDUCTOR
- added P?: CONN_8, symbol CONN_8
- added P? (x2): PWR-IN, symbol CONN_2
- added P? (x2): CONN_4, symbol CONN_4
- added Q? (x4): BC847, symbol NPN
- added Q? (x2): BC857, symbol PNP
- added Q?: MOS_N, symbol MOS_N
- added Q? (x3): MOS_P, symbol MOS_P
- added Q?: NPN, symbol NPN
- added R? (x4): 10k, symbol R
- added R? (x12): 30k, symbol R
- added R? (x2): 1k, symbol R
- added R? (x3): 50, symbol R
- added R? (x6): 500, symbol R
- added R? (x2): 100, symbol R
- C?: value 54u -> 1000u
Connections:
- net labels added: +6V, VCC, boost-fb, boost-out, boost-pwm, buck-fb, buck-out, buck-out-5v, buck-pwm, light, pwm-boost, pwm-buck, scl-int, scl-rpi, scl1, sda-int, sda-rpi, sda1, solar, solar-fb, vcc-test
- net labels removed: +24V, addr0, addr1, addr2, fw-upgrade, i-1-1, i-1-2, i-2-1, i-2-2, io-1-1, io-1-2, io-2-1, io-2-2, rx, scl, scl-ext, sda, sda-ext, sensor-1, sensor-2, synch, synch-ext, tx
- wire segments 162 -> 282
- no-connect marks 16 -> 24
Other:
- note added: "5V for powering raspberry-pi, \n3G modem, camera and so on..."
- note added: "Battery socket"
- note removed: "These Rs are not pullup but \njust current limiting. I2C bus \npullups are located near power \nsocket."
- moved on the sheet: C?, K?, P?, R?, X?, lsm?, stm?

Commit message: Designing scheme.
Parts:
- removed K?: CONN_3, symbol CONN_3
- removed P?: CONN_8, symbol CONN_8
- removed R?: 30k, symbol R
- added C11, C26, C6: 100n, symbol C
- added P4: PWR-IN, symbol CONN_2
- added P7: CONN_4, symbol CONN_4
- added Q10: BC847, symbol NPN
- added Q11: MOS_P, symbol MOS_P
- added R15, R19: 1, symbol R
- added R21, R22, R29, R30, R32, R50, R53: 30k, symbol R
- added R27: 10k, symbol R
- added R28: 65k, symbol R
- added R52: 500, symbol R
- added R54: 100, symbol R
- added U2: L293, symbol L293
- R16, R17, R18: renamed from R?; value 500 -> 1
- R33: renamed from R?; value 100 -> 500
- gave numbers to parts that had none: 94
Connections:
- net labels added: current-fb, just-power-source, moto-en, moto1, moto2, moto3, moto4, out1, out2, out3, out4
- net labels removed: VCC, boost-out, buck-out, pwm-boost, pwm-buck, scl1, sda1, vcc-test
- wire segments 282 -> 356
- no-connect marks 24 -> 17
Other:
- note added: "At zero frequency gain is (R28+R27)/R27.\nAim is to get +/-1.5Volts as current 2A.\nIf shunt resistors set resistance is 0.1Ohm\nthen they give 0.2V at 2A current.\nAmplification is 1.5/0.2 = 7.5.\nIf R27 = 10k.\nThen 7.5 = 1 + R28/10k.\nR28 = 10k * 6.5 = 65k."
- moved on the sheet: D3, D5, D6, R44, R45

Commit message: Planning board...
Parts:
- removed R2, R5: 10k, symbol R
- added EEPROM?: 24LC16B, symbol 24LC16B
Connections:
- wire segments 356 -> 358
Other:
- note added: "No pullups here as there are on raspberry-pi."

Commit message: Designing board.
Parts:
- added TC1: TC1047A, symbol TC1047A
- gave numbers to parts that had none: 1
Connections:
- net labels added: v-temp
- wire segments 358 -> 362
- no-connect marks 17 -> 16
Other:
- note added: "3.3V buck scheme for powering MCU."
- note added: "Analog \ntemperature\nsensor"
- note added: "Boost scheme for accumulator charging."
- note added: "Chassis motors control cheme."
- note added: "EEPROM"
- note added: "Indicator LEDs for debugging."
- note added: "Jumper here tells MCU to never turn 5V \nconverter off."
- note added: "Powerful LED on/off."
- note added: "Powerful buck scheme for 5V generation."
